File: ChillyCart.kicad_sch (KiCad schematic)
At the start: 14 parts, among them J1 GameBoy_GamePak_DMG-09, J2 USB_C_Receptacle_USB2.0_16P, U1 TXB0108PW, U2 TXB0108PW, U3 TXB0108PW, U4 RP2350_80QFN

Commit message: Added psram,flash,rtc,sd
Parts:
- added BT1: Battery_Cell, Battery:BatteryHolder_Keystone_103_1x20mm, symbol Device:Battery_Cell
- added C10, C9: 15p, Capacitor_SMD:C_0402_1005Metric, symbol Device:C
- added C11, C13, C14, C15, C16, C17, C18, C19, C20, C21, C25, C27: 100n, Capacitor_SMD:C_0402_1005Metric, symbol Device:C
- added C12: DNF, Capacitor_SMD:C_0402_1005Metric, symbol Device:C
- added C22, C23: 4.7u, RP2350_80QFN_minimal:C_0402_1005Metric_small_pads, symbol Device:C
- added C24, C26: 4.7u, Capacitor_SMD:C_0402_1005Metric, symbol Device:C
- added C28, C7: 10u, Capacitor_SMD:C_0805_2012Metric, symbol Device:C
- added J3: Micro_SD_Card_Det1, kicad-open-modules:TF-015, symbol Connector:Micro_SD_Card_Det1
- added L1: 3.3u, RP2350_80QFN_minimal:L_pol_2016, symbol Device:L
- added R10, R11: 27, Resistor_SMD:R_0402_1005Metric, symbol Device:R
- added R3: 1k, Resistor_SMD:R_0402_1005Metric, symbol Device:R
- added R4, R6, R7, R8: DNF, Resistor_SMD:R_0402_1005Metric, symbol Device:R
- added R5: 0, Resistor_SMD:R_0402_1005Metric, symbol Device:R
- added R9: 33, Resistor_SMD:R_0402_1005Metric, symbol Device:R
- added U5: AMS1117-3.3, Package_TO_SOT_SMD:SOT-223-3_TabPin2, symbol Regulator_Linear:AMS1117-3.3
- added U6: W25Q128JVS, Package_SO:SOIC-8_5.23x5.23mm_P1.27mm, symbol Memory_Flash:W25Q128JVS
- added U7: DNF, Package_SO:SOIC-8_5.23x5.23mm_P1.27mm, symbol Memory_Flash:W25Q128JVS
- added U8: MCP7940N-xMNY, Package_DFN_QFN:DFN-8-1EP_3x2mm_P0.5mm_EP1.36x1.46mm, symbol Timer_RTC:MCP7940N-xMNY
- added Y1: ABM8-272-T3, Crystal:Crystal_SMD_3225-4Pin_3.2x2.5mm, symbol Device:Crystal_GND24
Connections:
- net +3V3: now also U4.15 (IOVDD), U4.24 (IOVDD), U4.29 (IOVDD), U4.41 (IOVDD), U4.5 (IOVDD), U4.50 (IOVDD), U4.59 (ADC_AVDD), U4.60 (IOVDD), U4.64 (VREG_VIN), U4.68 (USB_OTP_VDD), U4.69 (QSPI_IOVDD), U4.76 (IOVDD), C11.1, C12.1, C13.1, C14.1, C15.1, C16.1, C17.1, C18.1, C19.1, C20.1, C21.1, C22.1, C7.1, R7.1, R8.1, R9.1, U5.2 (VO), U6.8 (VCC), U7.8 (VCC)
- net GND: now also U4.62 (VREG_PGND), U4.81 (GND), C10.2, C11.2, C12.2, C13.2, C14.2, C15.2, C16.2, C17.2, C18.2, C19.2, C20.2, C21.2, C22.2, C23.2, C24.2, C25.2, C26.2, C27.2, C28.2, C7.2, C9.2, U5.1 (GND), U6.4 (GND), U7.4 (GND), Y1.2, Y1.4
- net USB_D+: now also R10.1; no longer U4.67 (USB_DP)
- net USB_D-: now also R11.1; no longer U4.66 (USB_DM)
- net VCC: now also C28.1, U5.3 (VI)
- net +1V1: now reaches U4.10 (DVDD)
- net +1V1: now also U4.32 (DVDD), U4.51 (DVDD), U4.65 (VREG_FB), C23.1, C25.1, C26.1, C27.1, L1.1
- net VREG_AVDD: now reaches U4.61 (VREG_AVDD)
- net VREG_AVDD: now also C24.1, R9.2
- net VREG_LX: now reaches U4.63 (VREG_LX)
- net VREG_LX: now also L1.2
- net QSPI_SD3: now reaches U4.70 (QSPI_SD3)
- net QSPI_SD3: now also U6.7 (IO3), U7.7 (IO3)
- net QSPI_SCLK: now reaches U4.71 (QSPI_SCLK)
- net QSPI_SCLK: now also U6.6 (CLK), U7.6 (CLK)
- net QSPI_SD0: now reaches U4.72 (QSPI_SD0)
- net QSPI_SD0: now also U6.5 (DI(IO0)), U7.5 (DI(IO0))
- net QSPI_SD2: now reaches U4.73 (QSPI_SD2)
- net QSPI_SD2: now also U6.3 (IO2), U7.3 (IO2)
- net QSPI_SD1: now reaches U4.74 (QSPI_SD1)
- net QSPI_SD1: now also U6.2 (DO(IO1)), U7.2 (DO(IO1))
- net QSPI_SS: now reaches U4.75 (QSPI_SS)
- net QSPI_SS: now also R5.1
- new net: C10.1, R3.2, Y1.3
- new net: R10.2, U4.67 (USB_DP)
- new net: R11.2, U4.66 (USB_DM)
- new net FLASH2_SS: R6.2, R8.2, U7.1 (~{CS})
- new net FLASH_SS: R4.2, R5.2, R7.2, U6.1 (~{CS})
- new net GPIO0: R4.1, R6.1
- new net XIN: C9.1, Y1.1
- new net XOUT: R3.1
Other:
- note added: "12MHz Crystal"
- note added: "PSRAM"
- note added: "Primary Flash"
- moved on the sheet: U4

Commit message: Add IMU, power mux and cleanup schematic
Parts:
- removed BT1: Battery_Cell, Battery:BatteryHolder_Keystone_103_1x20mm, symbol Device:Battery_Cell
- removed U8: MCP7940N-xMNY, Package_DFN_QFN:DFN-8-1EP_3x2mm_P0.5mm_EP1.36x1.46mm, symbol Timer_RTC:MCP7940N-xMNY
- added C29, C8: 100nF, Capacitor_SMD:C_0603_1608Metric_Pad1.08x0.95mm_HandSolder, symbol Device:C
- added C30, C33: 100nF, Capacitor_SMD:C_0603_1608Metric, symbol Device:C
- added C31, C32: 7pF, Capacitor_SMD:C_0603_1608Metric, symbol Device:C
- added C34: 47uF, Capacitor_SMD:C_0805_2012Metric, symbol Device:C
- added C35: 10u, Capacitor_SMD:C_0805_2012Metric, symbol Device:C
- added C36: 100n, Capacitor_SMD:C_0805_2012Metric, symbol Device:C
- added J4: Conn_01x02_Socket, TestPoint:TestPoint_2Pads_Pitch2.54mm_Drill0.8mm, symbol Connector:Conn_01x02_Socket
- added R12: 10k, Resistor_SMD:R_0603_1608Metric, symbol Device:R
- added R13: 470R, symbol Device:R
- added R14, R15: 1k, Resistor_SMD:R_0402_1005Metric, symbol Device:R
- added U10: MCP7940N-x/ST, Package_SO:TSSOP-8_4.4x3mm_P0.65mm, symbol Timer_RTC:MCP7940N-xST
- added U11: LSM6DS3, Package_LGA:LGA-14_3x2.5mm_P0.5mm_LayoutBorder3x4y, symbol Sensor_Motion:LSM6DS3
- added U8: TPS2111A, Package_SO:TSSOP-8_4.4x3mm_P0.65mm, symbol sc64v2:TPS2111A
- added U9: TXB0108PW, Package_SO:TSSOP-20_4.4x6.5mm_P0.65mm, symbol Logic_LevelTranslator:TXS0108EPW
- added Y2: FC-135, Crystal:Crystal_SMD_3215-2Pin_3.2x1.5mm, symbol Device:Crystal
Connections:
- net XIN is gone; now on an unnamed net: C9.1, Y1.1
- net XOUT is gone; now on an unnamed net: R3.1
- net +3V3: now also J3.4 (VDD), C30.1, C33.1, C34.1, C36.1, C8.2, R12.1, U10.8 (VCC), U11.12 (CS), U11.5 (VDDIO), U11.8 (VDD), U9.2 (VCCA)
- net ADDR0: now also U2.12 (B8); no longer U2.1 (A1)
- net ADDR1: now also U2.13 (B7); no longer U2.3 (A2)
- net ADDR10: now also U3.14 (B6); no longer U3.4 (A3)
- net ADDR11: now also U3.15 (B5); no longer U3.5 (A4)
- net ADDR12: now also U3.16 (B4); no longer U3.6 (A5)
- net ADDR13: now also U3.17 (B3); no longer U3.7 (A6)
- net ADDR14: now also U3.18 (B2); no longer U3.8 (A7)
- net ADDR15: now also U3.20 (B1); no longer U3.9 (A8)
- net ADDR2: now also U2.14 (B6); no longer U2.4 (A3)
- net ADDR3: now also U2.15 (B5); no longer U2.5 (A4)
- net ADDR4: now also U2.16 (B4); no longer U2.6 (A5)
- net ADDR5: now also U2.17 (B3); no longer U2.7 (A6)
- net ADDR6: now also U2.18 (B2); no longer U2.8 (A7)
- net ADDR7: now also U2.20 (B1); no longer U2.9 (A8)
- net ADDR8: now also U3.12 (B8); no longer U3.1 (A1)
- net ADDR9: now also U3.13 (B7); no longer U3.3 (A2)
- net DATA0: now also U1.12 (B8); no longer U1.1 (A1)
- net DATA1: now also U1.13 (B7); no longer U1.3 (A2)
- net DATA2: now also U1.14 (B6); no longer U1.4 (A3)
- net DATA3: now also U1.15 (B5); no longer U1.5 (A4)
- net DATA4: now also U1.16 (B4); no longer U1.6 (A5)
- net DATA5: now also U1.17 (B3); no longer U1.7 (A6)
- net DATA6: now also U1.18 (B2); no longer U1.8 (A7)
- net DATA7: now also U1.20 (B1); no longer U1.9 (A8)
- net GND: now also J3.10 (SHIELD), J3.6 (VSS), C29.1, C30.2, C31.2, C32.1, C33.2, C34.2, C35.2, C36.2, C8.1, J4.2 (Pin_2), R13.2, R15.2, U10.4 (VSS), U11.2 (SDX), U11.3 (SCX), U11.6 (GND), U11.7 (GND), U8.2 (D1), U8.5 (GND), U9.11 (GND)
- net GPIO0: now also U4.77 (GPIO0)
- net RP_ADDR0: now also U2.9 (A8), U4.78 (GPIO1); no longer U2.20 (B1), U4.77 (GPIO0)
- net RP_ADDR1: now also U2.8 (A7), U4.79 (GPIO2); no longer U2.18 (B2), U4.78 (GPIO1)
- net RP_ADDR10: now also U3.7 (A6), U4.9 (GPIO11); no longer U3.17 (B3), U4.8 (GPIO10)
- net RP_ADDR11: now also U3.6 (A5), U4.11 (GPIO12); no longer U3.16 (B4), U4.9 (GPIO11)
- net RP_ADDR12: now also U3.5 (A4), U4.12 (GPIO13); no longer U3.15 (B5), U4.11 (GPIO12)
- net RP_ADDR13: now also U3.4 (A3), U4.13 (GPIO14); no longer U3.14 (B6), U4.12 (GPIO13)
- net RP_ADDR14: now also U3.3 (A2), U4.14 (GPIO15); no longer U3.13 (B7), U4.13 (GPIO14)
- net RP_ADDR15: now also U3.1 (A1), U4.16 (GPIO16); no longer U3.12 (B8), U4.14 (GPIO15)
- net RP_ADDR2: now also U2.7 (A6), U4.80 (GPIO3); no longer U2.17 (B3), U4.79 (GPIO2)
- net RP_ADDR3: now also U2.6 (A5), U4.1 (GPIO4); no longer U2.16 (B4), U4.80 (GPIO3)
- net RP_ADDR4: now also U2.5 (A4), U4.2 (GPIO5); no longer U2.15 (B5), U4.1 (GPIO4)
- net RP_ADDR5: now also U2.4 (A3), U4.3 (GPIO6); no longer U2.14 (B6), U4.2 (GPIO5)
- net RP_ADDR6: now also U2.3 (A2), U4.4 (GPIO7); no longer U2.13 (B7), U4.3 (GPIO6)
- net RP_ADDR7: now also U2.1 (A1), U4.6 (GPIO8); no longer U2.12 (B8), U4.4 (GPIO7)
- net RP_ADDR8: now also U3.9 (A8), U4.7 (GPIO9); no longer U3.20 (B1), U4.6 (GPIO8)
- net RP_ADDR9: now also U3.8 (A7), U4.8 (GPIO10); no longer U3.18 (B2), U4.7 (GPIO9)
- net RP_DATA0: now also U1.9 (A8), U4.17 (GPIO17); no longer U1.20 (B1), U4.16 (GPIO16)
- net RP_DATA1: now also U1.8 (A7), U4.18 (GPIO18); no longer U1.18 (B2), U4.17 (GPIO17)
- net RP_DATA2: now also U1.7 (A6), U4.19 (GPIO19); no longer U1.17 (B3), U4.18 (GPIO18)
- net RP_DATA3: now also U1.6 (A5), U4.20 (GPIO20); no longer U1.16 (B4), U4.19 (GPIO19)
- net RP_DATA4: now also U1.5 (A4), U4.21 (GPIO21); no longer U1.15 (B5), U4.20 (GPIO20)
- net RP_DATA5: now also U1.4 (A3), U4.22 (GPIO22); no longer U1.14 (B6), U4.21 (GPIO21)
- net RP_DATA6: now also U1.3 (A2), U4.23 (GPIO23); no longer U1.13 (B7), U4.22 (GPIO22)
- net RP_DATA7: now also U1.1 (A1), U4.25 (GPIO24); no longer U1.12 (B8), U4.23 (GPIO23)
- net USB_VCC: now also C35.1, R14.1, U8.8 (IN1)
- net CLK: now reaches J1.2 (PHI)
- net CLK: now also U9.1 (A1)
- net WR: now reaches J1.3 (~{WR})
- net WR: now also U9.3 (A2)
- net RST: now reaches J1.30 (~{RST})
- net RST: now also U9.6 (A5)
- net RD: now reaches J1.4 (~{RD})
- net RD: now also U9.4 (A3)
- net CS: now reaches J1.5 (~{CS})
- net CS: now also U9.5 (A4)
- net RP_CLK: now reaches U4.26 (GPIO25)
- net RP_CLK: now also U9.20 (B1)
- net RP_WR: now reaches U4.27 (GPIO26)
- net RP_WR: now also U9.18 (B2)
- net RP_RD: now reaches U4.28 (GPIO27)
- net RP_RD: now also U9.17 (B3)
- net RP_CS: now reaches U4.36 (GPIO28)
- net RP_CS: now also U9.16 (B4)
- net RP_RST: now reaches U4.37 (GPIO29)
- net RP_RST: now also U9.15 (B5)
- net RTC_SDA: now reaches U4.38 (GPIO30)
- net RTC_SDA: now also U10.5 (SDA)
- net RTC_SCL: now reaches U4.39 (GPIO31)
- net RTC_SCL: now also U10.6 (SCL)
- net SD_MISO: now reaches U4.40 (GPIO32)
- net SD_MISO: now also J3.7 (DAT0)
- net SD_DAT3: now reaches U4.42 (GPIO33)
- net SD_DAT3: now also J3.2 (DAT3/CD)
- net SD_CLK: now reaches U4.43 (GPIO34)
- net SD_CLK: now also J3.5 (CLK)
- net SD_MOSI: now reaches U4.44 (GPIO35)
- net SD_MOSI: now also J3.3 (CMD)
- net IMU_SDA: now reaches U4.45 (GPIO36)
- net IMU_SDA: now also U11.14 (SDA)
- net IMU_SCL: now reaches U4.46 (GPIO37)
- net IMU_SCL: now also U11.13 (SCL)
- net SD_DET: now reaches U4.47 (GPIO38)
- net SD_DET: now also J3.9 (DET), R12.2
- net RP_POWER: now reaches U4.48 (GPIO39)
- net RP_POWER: now also U9.14 (B6)
- removed net POWER_GOOD: U1.10 (OE), U2.10 (OE), U3.10 (OE)
- net VCC renamed +5V_CART
- net +5V_CART: now also C29.2, U8.6 (IN2), U9.19 (VCCB), U9.7 (A6); no longer C28.1, U5.3 (VI)
- new net: C32.2, U10.2 (X2), Y2.2
- new net: C31.1, U10.1 (X1), Y2.1
- new net: J4.1 (Pin_1), U10.3 (VBAT)
- new net: R14.2, R15.1, U8.3 (VSNS)
- new net: R13.1, U8.4 (ILM)
- new net: C28.1, U5.3 (VI), U8.7 (OUT)
- no-connect marks 2 -> 13
Other:
- note added: "3.3 regulator"
- note added: "Cartridge connector"
- note added: "Flash"
- note added: "I2C1"
- note added: "IMU"
- note added: "MCU"
- note added: "Power"
- note added: "Power mux: prefer USB over GB power"
- note added: "RTC"
- note added: "SD Card"
- note added: "SPI0"
- note removed: "12MHz Crystal"
- note removed: "Primary Flash"
- moved on the sheet: C1, C10, C11, C12, C13, C14, C15, C16, C17, C18, C19, C2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

Commit message: Add debug connectors and push button, fix ERC errors
Parts:
- added J5: Conn_01x02_Socket, TestPoint:TestPoint_2Pads_Pitch2.54mm_Drill0.8mm, symbol Connector:Conn_01x02_Socket
- added J7: Conn_01x07_Socket, symbol Connector:Conn_01x07_Socket
- added SW1: SW_Push, symbol Switch:SW_Push
Connections:
- net +3V3: now also U1.10 (OE), U2.10 (OE), U3.10 (OE), U4.35 (RUN), U9.10 (OE)
- net GND: now also SW1.2
- net +VBAT: now reaches J4.1 (Pin_1), U10.3 (VBAT)
- net at U4.33 (SWCLK): now also J5.2 (Pin_2)
- net at U4.34 (SWD): now also J5.1 (Pin_1)
- net at U4.49 (GPIO40_ADC0): now also SW1.1
- net at U4.52 (GPIO41_ADC1): now also J7.1 (Pin_1)
- net at U4.53 (GPIO42_ADC2): now also J7.2 (Pin_2)
- net at U4.54 (GPIO43_ADC3): now also J7.3 (Pin_3)
- net at U4.55 (GPIO44_ADC4): now also J7.4 (Pin_4)
- net at U4.56 (GPIO45_ADC5): now also J7.5 (Pin_5)
- net at U4.57 (GPIO46_ADC6): now also J7.6 (Pin_6)
- net at U4.58 (GPIO47_ADC7): now also J7.7 (Pin_7)
- no-connect marks 13 -> 14
Other:
- moved on the sheet: C1, C11, C3, C5, C8, R6, R7, R8, U6

Commit message: Initial routing
Parts:
- C1, C2, C29, C3, C4, C5, C6, C8: footprint Capacitor_SMD:C_0603_1608Metric_Pad1.08x0.95mm_HandSolder -> Capacitor_SMD:C_0402_1005Metric_Pad0.74x0.62mm_HandSolder
- C10, C11, C12, C13, C14, C15, C16, C17, C18, C19, C20, C21, C24, C25, C26, C27, C9: footprint Capacitor_SMD:C_0402_1005Metric -> Capacitor_SMD:C_0402_1005Metric_Pad0.74x0.62mm_HandSolder
- C22, C23: footprint RP2350_80QFN_minimal:C_0402_1005Metric_small_pads -> Capacitor_SMD:C_0402_1005Metric_Pad0.74x0.62mm_HandSolder
- C28, C34, C35, C36, C7: footprint Capacitor_SMD:C_0805_2012Metric -> Capacitor_SMD:C_0402_1005Metric_Pad0.74x0.62mm_HandSolder
- C30, C31, C32, C33: footprint Capacitor_SMD:C_0603_1608Metric -> Capacitor_SMD:C_0402_1005Metric_Pad0.74x0.62mm_HandSolder
- R1, R10, R11, R14, R15, R2, R3, R4, R5, R6, R7, R8, R9: footprint Resistor_SMD:R_0402_1005Metric -> Resistor_SMD:R_0402_1005Metric_Pad0.72x0.64mm_HandSolder
- R12: footprint Resistor_SMD:R_0603_1608Metric -> Resistor_SMD:R_0402_1005Metric_Pad0.72x0.64mm_HandSolder
- R13: footprint (none) -> Resistor_SMD:R_0402_1005Metric_Pad0.72x0.64mm_HandSolder
- SW1: footprint (none) -> Button_Switch_SMD:SW_Push_1P1T_XKB_TS-1187A
Connections:
- net +5V_CART: now also U9.17 (B3); no longer U9.7 (A6)
- net CLK: now also U9.12 (B8); no longer U9.1 (A1)
- net CS: now also U9.15 (B5); no longer U9.5 (A4)
- net RD: now also U9.14 (B6); no longer U9.4 (A3)
- net RP_CLK: now also U4.37 (GPIO29), U9.9 (A8); no longer U4.26 (GPIO25), U9.20 (B1)
- net RP_CS: now also U4.27 (GPIO26), U9.6 (A5); no longer U4.36 (GPIO28), U9.16 (B4)
- net RP_POWER: now also U9.4 (A3); no longer U9.14 (B6)
- net RP_RD: now also U9.7 (A6); no longer U9.17 (B3)
- net RP_RST: now also U4.26 (GPIO25), U9.5 (A4); no longer U4.37 (GPIO29), U9.15 (B5)
- net RP_WR: now also U4.36 (GPIO28), U9.8 (A7); no longer U4.27 (GPIO26), U9.18 (B2)
- net RST: now also U9.16 (B4); no longer U9.6 (A5)
- net WR: now also U9.13 (B7); no longer U9.3 (A2)
- no-connect marks 14 -> 15

Commit message: Finish routingn
Parts:
- removed J7: Conn_01x07_Socket, symbol Connector:Conn_01x07_Socket
- added J6: Conn_01x02_Socket, TestPoint:TestPoint_2Pads_Pitch2.54mm_Drill0.8mm, symbol Connector:Conn_01x02_Socket
- added J7: Conn_01x09_Socket, Connector_PinHeader_1.00mm:PinHeader_1x09_P1.00mm_Vertical, symbol Connector:Conn_01x09_Socket
- added R16: 1k, Resistor_SMD:R_0402_1005Metric_Pad0.72x0.64mm_HandSolder, symbol Device:R
Connections:
- net +3V3: now also J7.8 (Pin_8)
- net GND: now also J6.2 (Pin_2), J7.9 (Pin_9)
- net QSPI_SS: now also R16.1
- net at U4.52 (GPIO41_ADC1): now also J7.1 (Pin_1)
- net at U4.53 (GPIO42_ADC2): now also J7.2 (Pin_2)
- net at U4.54 (GPIO43_ADC3): now also J7.3 (Pin_3)
- net at U4.55 (GPIO44_ADC4): now also J7.4 (Pin_4)
- net at U4.56 (GPIO45_ADC5): now also J7.5 (Pin_5)
- net at U4.57 (GPIO46_ADC6): now also J7.6 (Pin_6)
- net at U4.58 (GPIO47_ADC7): now also J7.7 (Pin_7)
- new net ~{USB_BOOT}: J6.1 (Pin_1), R16.2
